File: Alaris - Hardware/AlarisV1.0/ADA.kicad_sch (KiCad schematic)
At the start: 25 parts, among them J2 Screw_Term, Q3 CMA-4544PF-W, U18 MAX4466EXK, U3 INA333xxDGK, U7 LM358D, U9 INA333xxDGK

Commit message: Desenvolvimento da PCB
Parts:
- removed J2: Screw_Term, symbol Connector:Screw_Terminal_01x02
- removed Q3: CMA-4544PF-W, Adafruit MAX4466 Mic Amp:ELECTRET_9.7, symbol Adafruit MAX4466 Mic Amp-eagle-import:ELECTRET
- removed U7: LM358D, LM358D:SOIC127P599X175-8N, symbol LM358D:LM358D
- added C29, C44, C45, C46: 100nF, Capacitor_SMD:C_0603_1608Metric_Pad1.08x0.95mm_HandSolder, symbol Device:C
- added J11, J12, J13, J14: Conn_01x02_Pin, Connector_JST:JST_EH_B2B-EH-A_1x02_P2.50mm_Vertical, symbol Connector:Conn_01x02_Pin
- added MK1: CMC-6022-42P, Footprint:Mic6022, symbol Mic6022:CMC-6022-42P
- added R12: 1k, Resistor_SMD:R_0603_1608Metric_Pad0.98x0.95mm_HandSolder, symbol Device:R
- added R13, R50, R51, R52: 10k, Resistor_SMD:R_0603_1608Metric_Pad0.98x0.95mm_HandSolder, symbol Device:R
- added U1, U7: TL084, Package_SO:SOIC-14_3.9x8.7mm_P1.27mm, symbol Amplifier_Operational:TL084
- R25, R26, R27, R28, R29, R30: footprint Adafruit MAX4466 Mic Amp:0805 -> Resistor_SMD:R_0603_1608Metric_Pad0.98x0.95mm_HandSolder
- RV1, RV2: footprint (none) -> Potentiometer_SMD:Potentiometer_Bourns_TC33X_Vertical
- U11: footprint (none) -> FootPrintsMeus:MPS20N0040D
- VR3: renamed from VR1; footprint Adafruit MAX4466 Mic Amp:TRIMPOT_BOURNS_TC33X-2 -> Potentiometer_SMD:Potentiometer_Bourns_TC33X_Vertical
Connections:
- net +3.3V: now also C44.2, C45.2, C46.2, J11.2 (Pin_2), J12.2 (Pin_2), J13.2 (Pin_2), J14.2 (Pin_2), U1.4 (V+), U7.4 (V+)
- net AGND: now also MK1.GND
- net A_STG: now also U7.3 (+)
- net A_mic: now also U1.10 (+)
- net A_pitot: now also U1.5 (+)
- net GND: now also C29.2, C44.1, C45.1, C46.1, R13.2, R50.2, R51.2, R52.2, U1.11 (V-), U7.11 (V-)
- net at C18.1 (P$1), R26.1: now also MK1.OUT
- net SG_N renamed SG1_N
- net SG1_N: now also J14.1 (Pin_1)
- net SG_P renamed SG1_P
- new net A_DAil: J11.1 (Pin_1), R50.1, U7.12 (+)
- new net A_DProf: J12.1 (Pin_1), R51.1, U7.10 (+)
- new net A_DRud: J13.1 (Pin_1), R52.1, U7.5 (+)
- new net BattVA: C29.1, R12.2, R13.1, U1.12 (+)
- new net BatteryVoltage: U1.13 (-), U1.14
- new net DefAil: U7.13 (-), U7.14
- new net DefProf: U7.8, U7.9 (-)
- new net DefRud: U7.6 (-), U7.7
- new net Mic: U1.8, U1.9 (-)
- new net STG1: U7.1, U7.2 (-)
- new net Vin: R12.1
- new net WarmUP_mode: U1.3 (+)
- new net WarmUP_mode_OP: U1.1, U1.2 (-)
- new net pitot: U1.6 (-), U1.7
Other:
- note added: "Buffer_2"
- note added: "Deflexão Aileron"
- note added: "Deflexão Leme"
- note added: "Deflexão Profundor"
- note added: "Tensão bateria"
