File: Alaris - Hardware/AlarisV1.0/PSN.kicad_sch (KiCad schematic)
At the start: 36 parts, among them Q1 SI2302, Q2 BC856W, U12 LM3914N, U14 LP2985-3.3, U6 AMS1117-3.3

Commit message: Hardware and Software
Hardware: adição da proteção contra polaridade reversa
Software: Adição dos arquivos iniciais de projeto do LDIN
Parts:
- added D6: 12V, symbol Device:D_Schottky
- added F1: 3A, Fuse:Fuse_0603_1608Metric_Pad1.05x0.95mm_HandSolder, symbol Device:Fuse
- added Q4: FDS4559, Package_SO:SOIC-8_3.9x4.9mm_P1.27mm, symbol Transistor_FET:FDS4559
- added R49: 100k, Resistor_SMD:R_0603_1608Metric_Pad0.98x0.95mm_HandSolder, symbol Device:R
Connections:
- net +BATT: now also Q4.5 (D), Q4.6 (D); no longer S1.2
- net GND: now also R49.2
- new net: D6.2 (A), Q4.4 (G), R49.1
- new net: D6.1 (K), F1.2, Q4.3 (1)
- new net: Q4.7 (D), Q4.8 (D)
- new net VBUS: F1.1, S1.2
Other:
- note added: "Reverse polarity & protection"
- moved on the sheet: BAR1, C8, D4, FB1, FB2, Q2, R20, R21, R22, R23, R24, R4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

Commit message: Desenvolvimento da PCB
Parts:
- removed BAR1: HLCP-J100_2, Display:HLCP-J100, symbol LED:HLCP-J100_2
- removed C29: 100nF, Capacitor_SMD:C_0603_1608Metric_Pad1.08x0.95mm_HandSolder, symbol Device:C
- removed C8: 5k, symbol Device:C_Trim
- removed D4: 1N4148WT, Diode_SMD:D_SOD-523, symbol Diode:1N4148WT
- removed Q2: BC856W, Package_TO_SOT_SMD:SOT-323_SC-70, symbol Transistor_BJT:BC856W
- removed R12: 1k, Resistor_SMD:R_0603_1608Metric_Pad0.98x0.95mm_HandSolder, symbol Device:R
- removed R13: 10k, Resistor_SMD:R_0603_1608Metric_Pad0.98x0.95mm_HandSolder, symbol Device:R
- removed R20: 27k, Resistor_SMD:R_0603_1608Metric_Pad0.98x0.95mm_HandSolder, symbol Device:R
- removed R21: 15k, Resistor_SMD:R_0603_1608Metric_Pad0.98x0.95mm_HandSolder, symbol Device:R
- removed R22: 120, Resistor_SMD:R_0603_1608Metric_Pad0.98x0.95mm_HandSolder, symbol Device:R
- removed R23: 2k2, Resistor_SMD:R_0603_1608Metric_Pad0.98x0.95mm_HandSolder, symbol Device:R
- removed R24: 620, Resistor_SMD:R_0603_1608Metric_Pad0.98x0.95mm_HandSolder, symbol Device:R
- removed U12: LM3914N, Package_DIP:DIP-18_W7.62mm, symbol Driver_LED:LM3914N
- added C36: 1uF, Capacitor_SMD:C_0603_1608Metric_Pad1.08x0.95mm_HandSolder, symbol Device:C
- added C38: 10nF, Capacitor_SMD:C_0603_1608Metric_Pad1.08x0.95mm_HandSolder, symbol Device:C
- added C39: 10uF, Capacitor_Tantalum_SMD:CP_EIA-3216-18_Kemet-A_Pad1.58x1.35mm_HandSolder, symbol Device:C_Polarized
- added C80: 2.2uF, Capacitor_SMD:C_0603_1608Metric_Pad1.08x0.95mm_HandSolder, symbol Device:C
- added J1: Conn_01x02_Pin, Connector_JST:JST_EH_B2B-EH-A_1x02_P2.50mm_Vertical, symbol Connector:Conn_01x02_Pin
- added R6, R9: 4k7, Resistor_SMD:R_0603_1608Metric_Pad0.98x0.95mm_HandSolder, symbol Device:R
- added U15: LP2985-3.3, Package_TO_SOT_SMD:SOT-23-5, symbol Regulator_Linear:LP2985-3.3
- C14: footprint (none) -> Capacitor_Tantalum_SMD:CP_EIA-3216-18_Kemet-A_Pad1.58x1.35mm_HandSolder
- C15: value 10uF -> 22uF; footprint (none) -> Capacitor_Tantalum_SMD:CP_EIA-3216-18_Kemet-A_Pad1.58x1.35mm_HandSolder
- D6: footprint (none) -> Diode_SMD:D_0603_1608Metric_Pad1.05x0.95mm_HandSolder
- FB1, FB2: footprint Adafruit MAX4466 Mic Amp:0805 -> Capacitor_SMD:C_0603_1608Metric_Pad1.08x0.95mm_HandSolder
- R3: footprint Resistor_SMD:R_0201_0603Metric_Pad0.64x0.40mm_HandSolder -> Resistor_SMD:R_0603_1608Metric_Pad0.98x0.95mm_HandSolder
Connections:
- net +3.3V: now also R6.1
- net +BATT: now also J1.1 (Pin_1)
- net 1.65V_Ref: now also R6.2, R9.1
- net GND: now also Q4.1 (S), C36.2, C38.2, C39.2, C80.2, J1.2 (Pin_2), R9.2, U15.2 (GND); no longer Q1.2 (S)
- net Vin: now also C36.1, U15.1 (VIN), U15.3 (ON/~{OFF})
- net WarmUP_mode: now also Q4.7 (D), Q4.8 (D); no longer Q1.3 (D)
- net at Q1.1 (G): no longer R17.1
- net at Q4.2 (G): now also R17.1
- new net: C38.1, U15.4 (BP)
- new net +3.3GPS: C39.1, C80.1, U15.5 (VOUT)
Other:
- moved on the sheet: C23, C37, C42, Q1, Q4A, R4, R5, U14
