File: Alaris - Hardware/AlarisV1.0/GNCN.kicad_sch (KiCad schematic)
At the start: 21 parts, among them J6 Header 4x2, SW5 SW_MEC_5G, SW6 SW_MEC_5G, U17 STM32F446RCTx, Y5 25MHz

Commit message: Desenvolvimento da PCB
Parts:
- removed SW5, SW6: SW_MEC_5G, symbol Switch:SW_MEC_5G
- added C1, C2: 22pF, Capacitor_SMD:C_0603_1608Metric_Pad1.08x0.95mm_HandSolder, symbol Device:C
- added C3, C4: 100nF, Capacitor_SMD:C_0603_1608Metric_Pad1.08x0.95mm_HandSolder, symbol Device:C
- added C5: 120nF, Capacitor_SMD:C_0603_1608Metric_Pad1.08x0.95mm_HandSolder, symbol Device:C
- added C6: 6.8nF, Capacitor_SMD:C_0603_1608Metric_Pad1.08x0.95mm_HandSolder, symbol Device:C
- added D10, D7, D8, D9: Verde, LED_SMD:LED_0603_1608Metric_Pad1.05x0.95mm_HandSolder, symbol Device:LED
- added R2: 10k, Resistor_SMD:R_0603_1608Metric_Pad0.98x0.95mm_HandSolder, symbol Device:R
- added R53, R54, R55, R56: 1k, Resistor_SMD:R_0603_1608Metric_Pad0.98x0.95mm_HandSolder, symbol Device:R
- added R63, R64: 4k7, Resistor_SMD:R_0603_1608Metric_Pad0.98x0.95mm_HandSolder, symbol Device:R
- added SW3, SW4: SW_Push, Footprint:SKRK, symbol Cleber:SW_Push
- added U2: BNO055, Package_LGA:LGA-28_5.2x3.8mm_P0.5mm, symbol Sensor_Motion:BNO055
- added Y1: 32k768, Crystal:Crystal_SMD_3215-2Pin_3.2x1.5mm, symbol Device:Crystal
- FB5: footprint (none) -> Capacitor_SMD:C_0603_1608Metric_Pad1.08x0.95mm_HandSolder
- R38, R39: footprint (none) -> Resistor_SMD:R_0603_1608Metric_Pad0.98x0.95mm_HandSolder
- Y5: footprint Crystal:Crystal_SMD_0603-4Pin_6.0x3.5mm_HandSoldering -> Crystal:Crystal_SMD_3225-4Pin_3.2x2.5mm
Connections:
- net +3.3VLN is gone; now on net +3.3V: FB5.1
- net DN_SWCLK is gone; now on net GN_SWCLK: R38.1
- net DN_SWDIO is gone; now on net GN_SWDIO: R39.1
- net PB2 is gone; now on net GN_PB2: R41.1
- net +3.3V: now also C4.1, C5.1, C6.1, R2.2, R63.1, R64.1, SW4.1, U2.28 (VDDIO), U2.3 (VDD)
- net GND: now also C1.2, C2.2, C3.2, C4.2, C5.2, C6.2, R53.1, R54.1, R55.1, R56.1, SW3.2, U2.15 (PIN15), U2.16 (PIN16), U2.18 (COM2), U2.2 (GND), U2.25 (GNDIO), U2.5 (PS1), U2.6 (PS0)
- net GN_BOOT0: now also SW4.2
- net GN_L_workingStatus: now also U17.11 (PC3), D10.2 (A); no longer U17.8 (PC0)
- net GN_NRST: now also SW3.1
- net GN_L_COM: now reaches U17.10 (PC2)
- net GN_L_COM: now also D9.2 (A)
- net GN_PWM_In5: now reaches U17.14 (PA0)
- net GN_PWM_O_T5_C3: now reaches U17.16 (PA2)
- net GN_PWM_O_T5_C4: now reaches U17.17 (PA3)
- net GN_PWM_In2: now reaches U17.21 (PA5)
- net GN_PWM_In3: now reaches U17.22 (PA6)
- net GN_PWM_O_T3_C3: now reaches U17.26 (PB0)
- net GN_PWM_O_T3_C4: now reaches U17.27 (PB1)
- net GN_PB2: now reaches U17.28 (PB2)
- net GN_PWM_O_T2_C3: now reaches U17.29 (PB10)
- net GN_PWM_O_T12_C1: now reaches U17.35 (PB14)
- net GN_PWM_O_T12_C2: now reaches U17.36 (PB15)
- net GN_PWM_In8: now reaches U17.37 (PC6)
- net GN_PWM_O_T8_C3: now reaches U17.39 (PC8)
- net GN_PWM_O_T8_C4: now reaches U17.40 (PC9)
- net GN_PWM_In1: now reaches U17.41 (PA8)
- net GN_SPI1_NSS: now reaches U17.50 (PA15)
- net GN_SPI1_SCK: now reaches U17.55 (PB3)
- net GN_SPI1_MISO: now reaches U17.56 (PB4)
- net GN_SPI1_MOSI: now reaches U17.57 (PB5)
- net GN_PWM_In4: now reaches U17.58 (PB6)
- net GN_SDA: now reaches U17.59 (PB7)
- net GN_SDA: now also R63.2, U2.20 (COM0)
- net GN_SLC: now reaches U17.61 (PB8)
- net GN_SLC: now also R64.2, U2.19 (COM1)
- net Addrs_Select: now reaches U17.62 (PB9)
- net Addrs_Select: now also U2.17 (COM3)
- net GN_L_Reading: now reaches U17.9 (PC1)
- net GN_L_Reading: now also D8.2 (A)
- new net: C2.1, U2.27 (XIN32), Y1.1
- new net: C1.1, U2.26 (XOUT32), Y1.2
- new net: D9.1 (K), R55.2
- new net: D10.1 (K), R56.2
- new net: R2.1, U2.11 (~{RESET})
- new net: C3.1, U2.9 (CAP)
- new net: D7.1 (K), R53.2
- new net: D8.1 (K), R54.2
- new net GN_L_AutoStatus: D7.2 (A), U17.8 (PC0)
- new net Int: U2.14 (INT)
Other:
- added sheet LevelShifter (LevelShifter.kicad_sch)
- added sheet PWM (PWM.kicad_sch)
- note added: "IMU1 (0x29)"
- moved on the sheet: C57, C58, C68, FB5, U17, Y5

Commit message: Mudanças GNCN
Adição do acelerômetro de backup
Mudanças no PWM read
Adição da comunicação entre núcleos utilizando SPI
Connections:
- net GND: now also U2.17 (COM3)
- net Addrs_Select: no longer names the net of U17.62 (PB9)
- net Addrs_Select: no longer U2.17 (COM3)
Other:
- moved on the sheet: C57, C58, C68, FB5, U17, Y5
